Commit message: Update urdf3.xacro

File: urdf/urdf3.xacro (robot description, xacro)
@@ -1,4 +1,4 @@
 <?xml version="1.0"?>
-<robot name="FYP2020-Swarm-Quadruped" xmlns:xacro="http://ros.org/wiki/xacro">
+<robot xmlns:xacro="http://ros.org/wiki/xacro" name="FYP2020-Swarm-Quadruped">
     <xacro:property name="shoul_len" value="0.035" />
     <xacro:property name="thigh_len" value="0.05" />
@@ -7,5 +7,5 @@
     <xacro:property name="feet_radius" value="0.0025"/>
     <xacro:property name="pi" value="3.1415" />
-    <xacro:property name="body_len" value="0.1" />
+    <xacro:property name="body_len" value="0.10" />
     <xacro:property name="body_width" value="0.05" />
     <xacro:property name="body_height" value="0.02" />
@@ -57,5 +57,5 @@
       <axis xyz="1 0 0"/>
       <parent link="base_link"/>
-      <child link="shoulder_link_lf}"/>
+      <child link="shoulder_link_lf"/>
     </joint>
     <link name="thigh_link_lf">
@@ -117,5 +117,5 @@
          <origin xyz="0 0 0" rpy="0 0 0"/>
          <geometry>
-            <cylinder radius="${feet_radius}"/>
+            <sphere radius="${feet_radius}"/>
          </geometry>
        </collision>
@@ -165,5 +165,5 @@
       <axis xyz="1 0 0"/>
       <parent link="base_link"/>
-      <child link="shoulder_link_rf}"/>
+      <child link="shoulder_link_rf"/>
     </joint>
     <link name="thigh_link_rf">
@@ -225,5 +225,5 @@
          <origin xyz="0 0 0" rpy="0 0 0"/>
          <geometry>
-            <cylinder radius="${feet_radius}"/>
+            <sphere radius="${feet_radius}"/>
          </geometry>
        </collision>
@@ -273,5 +273,5 @@
       <axis xyz="1 0 0"/>
       <parent link="base_link"/>
-      <child link="shoulder_link_lb}"/>
+      <child link="shoulder_link_lb"/>
     </joint>
     <link name="thigh_link_lb">
@@ -333,5 +333,5 @@
          <origin xyz="0 0 0" rpy="0 0 0"/>
          <geometry>
-            <cylinder radius="${feet_radius}"/>
+            <sphere radius="${feet_radius}"/>
          </geometry>
        </collision>
@@ -381,5 +381,5 @@
       <axis xyz="1 0 0"/>
       <parent link="base_link"/>
-      <child link="shoulder_link_rb}"/>
+      <child link="shoulder_link_rb"/>
     </joint>
     <link name="thigh_link_rb">
@@ -441,5 +441,5 @@
          <origin xyz="0 0 0" rpy="0 0 0"/>
          <geometry>
-            <cylinder radius="${feet_radius}"/>
+            <sphere radius="${feet_radius}"/>
          </geometry>
        </collision>

Commit message: Update urdf3.xacro

File: urdf/urdf3.xacro (robot description, xacro)
@@ -10,4 +10,6 @@
     <xacro:property name="body_width" value="0.05" />
     <xacro:property name="body_height" value="0.02" />
+    <xacro:property name="damping_value" value="10" />
+    <xacro:property name="friction_value" value="0.1" />
     <material name="red">
         <color rgba="255 0 0 1"/>
@@ -30,9 +32,15 @@
          <inertia ixx="1.0" ixy="0.0" ixz="0.0" iyy="1.0" iyz="0.0" izz="1.0" />
        </inertial>
+       <collision>
+         <origin xyz="0 0 0" rpy="0 0 0"/>
+         <geometry>
+            <box size="${body_len} ${body_width} ${body_height}" />
+         </geometry>
+       </collision>
     </link>
   <!--Left Front Leg-->
     <link name="shoulder_link_lf">
        <collision>
-         <origin xyz="0 0 0" rpy="0 0 0"/>
+         <origin rpy="${pi*0.5} 0 0" xyz="0 ${0.5*1.0*shoul_len} 0"/>
          <geometry>
             <cylinder radius="${link_radius}" length="${shoul_len}"/>
@@ -53,13 +61,14 @@
     </link>
     <joint name="shoulder_joint_lf" type="revolute">
-      <limit effort="1000.0" lower="${-0.5*pi}" upper="${0.5*pi}" velocity="0.5"/>
+      <limit effort="100.0" lower="${-0.5*pi}" upper="${0.5*pi}" velocity="0.5"/>
       <origin xyz="${0.5*body_len*1.0} ${1.0*0.005} 0"/>
       <axis xyz="1 0 0"/>
       <parent link="base_link"/>
       <child link="shoulder_link_lf"/>
+      <dynamics damping="${damping_value}" friction="${friction_value}"/>
     </joint>
     <link name="thigh_link_lf">
        <collision>
-         <origin xyz="0 0 0" rpy="0 0 0"/>
+         <origin rpy="0 0 0" xyz="0 0 ${-0.5*thigh_len}"/>
          <geometry>
             <cylinder radius="${link_radius}" length="${thigh_len}"/>
@@ -80,13 +89,14 @@
     </link>
     <joint name="elbow_joint_lf" type="revolute">
-      <limit effort="1000.0" lower="${-0.5*pi}" upper="${0.5*pi}" velocity="0.5"/>
+      <limit effort="100.0" lower="${-0.5*pi}" upper="${0.5*pi}" velocity="0.5"/>
       <origin xyz="0 ${1.0*shoul_len} 0"/>
       <axis xyz="0 1 0"/>
       <parent link="shoulder_link_lf"/>
       <child link="thigh_link_lf"/>
+      <dynamics damping="${damping_value}" friction="${friction_value}"/>
     </joint>
     <link name="shank_link_lf">
        <collision>
-         <origin xyz="0 0 0" rpy="0 0 0"/>
+         <origin rpy="0 0 0" xyz="0 0 ${-0.5*shank_len}"/>
          <geometry>
             <cylinder radius="${link_radius}" length="${shank_len}"/>
@@ -107,9 +117,10 @@
     </link>
     <joint name="wrist_joint_lf" type="revolute">
-      <limit effort="1000.0" lower="${-0.5*pi}" upper="${0.5*pi}" velocity="0.5"/>
+      <limit effort="100.0" lower="${-0.5*pi}" upper="${0.5*pi}" velocity="0.5"/>
       <origin xyz="0 0 ${-thigh_len}"/>
       <axis xyz="0 1 0"/>
       <parent link="thigh_link_lf"/>
       <child link="shank_link_lf"/>
+      <dynamics damping="${damping_value}" friction="${friction_value}"/>
     </joint>
     <link name="feet_link_lf">
@@ -138,9 +149,10 @@
       <parent link="shank_link_lf"/>
       <child link="feet_link_lf"/>
+      <dynamics damping="${damping_value}" friction="${friction_value}"/>
     </joint>
   <!--Right Front Leg-->
     <link name="shoulder_link_rf">
        <collision>
-         <origin xyz="0 0 0" rpy="0 0 0"/>
+         <origin rpy="${pi*0.5} 0 0" xyz="0 ${0.5*-1.0*shoul_len} 0"/>
          <geometry>
             <cylinder radius="${link_radius}" length="${shoul_len}"/>
@@ -161,13 +173,14 @@
     </link>
     <joint name="shoulder_joint_rf" type="revolute">
-      <limit effort="1000.0" lower="${-0.5*pi}" upper="${0.5*pi}" velocity="0.5"/>
+      <limit effort="100.0" lower="${-0.5*pi}" upper="${0.5*pi}" velocity="0.5"/>
       <origin xyz="${0.5*body_len*1.0} ${-1.0*0.005} 0"/>
       <axis xyz="1 0 0"/>
       <parent link="base_link"/>
       <child link="shoulder_link_rf"/>
+      <dynamics damping="${damping_value}" friction="${friction_value}"/>
     </joint>
     <link name="thigh_link_rf">
        <collision>
-         <origin xyz="0 0 0" rpy="0 0 0"/>
+         <origin rpy="0 0 0" xyz="0 0 ${-0.5*thigh_len}"/>
          <geometry>
             <cylinder radius="${link_radius}" length="${thigh_len}"/>
@@ -188,13 +201,14 @@
     </link>
     <joint name="elbow_joint_rf" type="revolute">
-      <limit effort="1000.0" lower="${-0.5*pi}" upper="${0.5*pi}" velocity="0.5"/>
+      <limit effort="100.0" lower="${-0.5*pi}" upper="${0.5*pi}" velocity="0.5"/>
       <origin xyz="0 ${-1.0*shoul_len} 0"/>
       <axis xyz="0 1 0"/>
       <parent link="shoulder_link_rf"/>
       <child link="thigh_link_rf"/>
+      <dynamics damping="${damping_value}" friction="${friction_value}"/>
     </joint>
     <link name="shank_link_rf">
        <collision>
-         <origin xyz="0 0 0" rpy="0 0 0"/>
+         <origin rpy="0 0 0" xyz="0 0 ${-0.5*shank_len}"/>
          <geometry>
             <cylinder radius="${link_radius}" length="${shank_len}"/>
@@ -215,9 +229,10 @@
     </link>
     <joint name="wrist_joint_rf" type="revolute">
-      <limit effort="1000.0" lower="${-0.5*pi}" upper="${0.5*pi}" velocity="0.5"/>
+      <limit effort="100.0" lower="${-0.5*pi}" upper="${0.5*pi}" velocity="0.5"/>
       <origin xyz="0 0 ${-thigh_len}"/>
       <axis xyz="0 1 0"/>
       <parent link="thigh_link_rf"/>
       <child link="shank_link_rf"/>
+      <dynamics damping="${damping_value}" friction="${friction_value}"/>
     </joint>
     <link name="feet_link_rf">
@@ -246,9 +261,10 @@
       <parent link="shank_link_rf"/>
       <child link="feet_link_rf"/>
+      <dynamics damping="${damping_value}" friction="${friction_value}"/>
     </joint>
   <!--Left Back Leg-->
     <link name="shoulder_link_lb">
        <collision>
-         <origin xyz="0 0 0" rpy="0 0 0"/>
+         <origin rpy="${pi*0.5} 0 0" xyz="0 ${0.5*1.0*shoul_len} 0"/>
          <geometry>
             <cylinder radius="${link_radius}" length="${shoul_len}"/>
@@ -269,13 +285,14 @@
     </link>
     <joint name="shoulder_joint_lb" type="revolute">
-      <limit effort="1000.0" lower="${-0.5*pi}" upper="${0.5*pi}" velocity="0.5"/>
+      <limit effort="100.0" lower="${-0.5*pi}" upper="${0.5*pi}" velocity="0.5"/>
       <origin xyz="${0.5*body_len*-1.0} ${1.0*0.005} 0"/>
       <axis xyz="1 0 0"/>
       <parent link="base_link"/>
       <child link="shoulder_link_lb"/>
+      <dynamics damping="${damping_value}" friction="${friction_value}"/>
     </joint>
     <link name="thigh_link_lb">
        <collision>
-         <origin xyz="0 0 0" rpy="0 0 0"/>
+         <origin rpy="0 0 0" xyz="0 0 ${-0.5*thigh_len}"/>
          <geometry>
             <cylinder radius="${link_radius}" length="${thigh_len}"/>
@@ -296,13 +313,14 @@
     </link>
     <joint name="elbow_joint_lb" type="revolute">
-      <limit effort="1000.0" lower="${-0.5*pi}" upper="${0.5*pi}" velocity="0.5"/>
+      <limit effort="100.0" lower="${-0.5*pi}" upper="${0.5*pi}" velocity="0.5"/>
       <origin xyz="0 ${1.0*shoul_len} 0"/>
       <axis xyz="0 1 0"/>
       <parent link="shoulder_link_lb"/>
       <child link="thigh_link_lb"/>
+      <dynamics damping="${damping_value}" friction="${friction_value}"/>
     </joint>
     <link name="shank_link_lb">
        <collision>
-         <origin xyz="0 0 0" rpy="0 0 0"/>
+         <origin rpy="0 0 0" xyz="0 0 ${-0.5*shank_len}"/>
          <geometry>
             <cylinder radius="${link_radius}" length="${shank_len}"/>
@@ -323,9 +341,10 @@
     </link>
     <joint name="wrist_joint_lb" type="revolute">
-      <limit effort="1000.0" lower="${-0.5*pi}" upper="${0.5*pi}" velocity="0.5"/>
+      <limit effort="100.0" lower="${-0.5*pi}" upper="${0.5*pi}" velocity="0.5"/>
       <origin xyz="0 0 ${-thigh_len}"/>
       <axis xyz="0 1 0"/>
       <parent link="thigh_link_lb"/>
       <child link="shank_link_lb"/>
+      <dynamics damping="${damping_value}" friction="${friction_value}"/>
     </joint>
     <link name="feet_link_lb">
@@ -354,9 +373,10 @@
       <parent link="shank_link_lb"/>
       <child link="feet_link_lb"/>
+      <dynamics damping="${damping_value}" friction="${friction_value}"/>
     </joint>
   <!--Right Back Leg-->
     <link name="shoulder_link_rb">
        <collision>
-         <origin xyz="0 0 0" rpy="0 0 0"/>
+         <origin rpy="${pi*0.5} 0 0" xyz="0 ${0.5*-1.0*shoul_len} 0"/>
          <geometry>
             <cylinder radius="${link_radius}" length="${shoul_len}"/>
@@ -377,13 +397,14 @@
     </link>
     <joint name="shoulder_joint_rb" type="revolute">
-      <limit effort="1000.0" lower="${-0.5*pi}" upper="${0.5*pi}" velocity="0.5"/>
+      <limit effort="100.0" lower="${-0.5*pi}" upper="${0.5*pi}" velocity="0.5"/>
       <origin xyz="${0.5*body_len*-1.0} ${-1.0*0.005} 0"/>
       <axis xyz="1 0 0"/>
       <parent link="base_link"/>
       <child link="shoulder_link_rb"/>
+      <dynamics damping="${damping_value}" friction="${friction_value}"/>
     </joint>
     <link name="thigh_link_rb">
        <collision>
-         <origin xyz="0 0 0" rpy="0 0 0"/>
+         <origin rpy="0 0 0" xyz="0 0 ${-0.5*thigh_len}"/>
          <geometry>
             <cylinder radius="${link_radius}" length="${thigh_len}"/>
@@ -404,13 +425,14 @@
     </link>
     <joint name="elbow_joint_rb" type="revolute">
-      <limit effort="1000.0" lower="${-0.5*pi}" upper="${0.5*pi}" velocity="0.5"/>
+      <limit effort="100.0" lower="${-0.5*pi}" upper="${0.5*pi}" velocity="0.5"/>
       <origin xyz="0 ${-1.0*shoul_len} 0"/>
       <axis xyz="0 1 0"/>
       <parent link="shoulder_link_rb"/>
       <child link="thigh_link_rb"/>
+      <dynamics damping="${damping_value}" friction="${friction_value}"/>
     </joint>
     <link name="shank_link_rb">
        <collision>
-         <origin xyz="0 0 0" rpy="0 0 0"/>
+         <origin rpy="0 0 0" xyz="0 0 ${-0.5*shank_len}"/>
          <geometry>
             <cylinder radius="${link_radius}" length="${shank_len}"/>
@@ -431,9 +453,10 @@
     </link>
     <joint name="wrist_joint_rb" type="revolute">
-      <limit effort="1000.0" lower="${-0.5*pi}" upper="${0.5*pi}" velocity="0.5"/>
+      <limit effort="100.0" lower="${-0.5*pi}" upper="${0.5*pi}" velocity="0.5"/>
       <origin xyz="0 0 ${-thigh_len}"/>
       <axis xyz="0 1 0"/>
       <parent link="thigh_link_rb"/>
       <child link="shank_link_rb"/>
+      <dynamics damping="${damping_value}" friction="${friction_value}"/>
     </joint>
     <link name="feet_link_rb">
@@ -462,4 +485,5 @@
       <parent link="shank_link_rb"/>
       <child link="feet_link_rb"/>
+      <dynamics damping="${damping_value}" friction="${friction_value}"/>
     </joint>
   <!--gazebo plugin-->
