Commit message: Update fyp_newv2.urdf

File: fyp_newv2.urdf (robot description, URDF)
Before this commit: robot fyp_new, 18 links, 17 joints
Links:
- link base_link: geometry collision box size=0.16 0.16 0.08; visual mesh filename=package://fyp_quadruped/meshes/body/body.stl scale=0.001 0.001 0.001
- link feet_link_lb: mass None -> 0.05
- link feet_link_lf: mass None -> 0.05
- link feet_link_rb: mass None -> 0.05
- link feet_link_rf: mass None -> 0.05
- link shank_link_lb: geometry collision box size=0.03 0.05 0.13; visual mesh filename=package://fyp_quadruped/meshes/leg/shank.stl scale=0.001 0.001 0.001
- link shank_link_lf: geometry collision box size=0.03 0.05 0.13; visual mesh filename=package://fyp_quadruped/meshes/leg/shank.stl scale=0.001 0.001 0.001
- link shank_link_rb: geometry collision box size=0.03 0.05 0.13; visual mesh filename=package://fyp_quadruped/meshes/leg/shank.stl scale=0.001 0.001 0.001
- link shank_link_rf: geometry collision box size=0.03 0.05 0.13; visual mesh filename=package://fyp_quadruped/meshes/leg/shank.stl scale=0.001 0.001 0.001
- link shoulder_link_lb: geometry collision box size=0.07 0.09 0.03; visual mesh filename=package://fyp_quadruped/meshes/leg/shoulder.stl scale=0.001 0.001 0.001
- link shoulder_link_lf: geometry collision box size=0.07 0.09 0.03; visual mesh filename=package://fyp_quadruped/meshes/leg/shoulder.stl scale=0.001 0.001 0.001
- link shoulder_link_rb: geometry collision box size=0.07 0.09 0.03; visual mesh filename=package://fyp_quadruped/meshes/leg/shoulder.stl scale=0.001 0.001 0.001
- link shoulder_link_rf: geometry collision box size=0.07 0.09 0.03; visual mesh filename=package://fyp_quadruped/meshes/leg/shoulder.stl scale=0.001 0.001 0.001
- link thigh_link_lb: geometry collision box size=0.03 0.07 0.21; visual mesh filename=package://fyp_quadruped/meshes/leg/thigh.stl scale=0.001 0.001 0.001
- link thigh_link_lf: geometry collision box size=0.03 0.07 0.21; visual mesh filename=package://fyp_quadruped/meshes/leg/thigh.stl scale=0.001 0.001 0.001
- link thigh_link_rb: geometry collision box size=0.03 0.07 0.21; visual mesh filename=package://fyp_quadruped/meshes/leg/thigh.stl scale=0.001 0.001 0.001
- link thigh_link_rf: geometry collision box size=0.03 0.07 0.21; visual mesh filename=package://fyp_quadruped/meshes/leg/thigh.stl scale=0.001 0.001 0.001
Joints:
- joint ankle_joint_lb: origin xyz=-0.144 0.175 0.05 -> xyz=0.1204 0.195 0.025
- joint ankle_joint_lf: origin xyz=0.144 0.175 0.05 -> xyz=0.3696 0.195 0.025
- joint ankle_joint_rb: origin xyz=-0.144 -0.175 0.05 -> xyz=0.1204 -0.035 0.025
- joint ankle_joint_rf: origin xyz=0.144 -0.175 0.05 -> xyz=0.3696 -0.035 0.025

Commit message: Update fyp_newv2.urdf

File: fyp_newv2.urdf (robot description, URDF)
Before this commit: robot fyp_quadruped, 18 links, 17 joints
Joints:
- joint ankle_joint_lb: origin xyz=0.1204 0.195 0.025 -> xyz=0.1204 0.195 0.0
- joint ankle_joint_lf: origin xyz=0.3696 0.195 0.025 -> xyz=0.3696 0.195 0.0
- joint ankle_joint_rb: origin xyz=0.1204 -0.035 0.025 -> xyz=0.1204 -0.035 0.0
- joint ankle_joint_rf: origin xyz=0.3696 -0.035 0.025 -> xyz=0.3696 -0.035 0.0
- joint base_link_to_base_inertia: origin xyz=0.0 0.0 0.0 rpy=0 0 0 -> xyz=0.0 0.0 0.2416 rpy=0 0 0
